Commit message: feat: add full Gazebo simulation integration with custom sticker workcell world and MoveIt 2 launch pipeline

File: src/Robot_to_URDF_New_Pakka_description/urdf/Robot_to_URDF_New_Pakka.urdf.xacro (robot description, xacro)
@@ -1,4 +1,7 @@
 <?xml version="1.0"?>
 <robot xmlns:xacro="http://www.ros.org/wiki/xacro" name="Robot_to_URDF_New_Pakka">
+  <!-- Arguments for simulation and hardware switching -->
+  <xacro:arg name="use_gazebo" default="false"/>
+  <xacro:arg name="gazebo_controllers" default="$(find kerabot_moveit_config)/config/ros2_controllers.yaml"/>
   <!-- Materials (shared across all assemblies) -->
   <material name="Steel">
@@ -17,8 +20,4 @@
   <xacro:Robot_Assembly_URDF_New prefix=""/>
   <!-- Mount joints (cross-assembly connections) -->
-  <!-- These define how assemblies connect to each other. -->
-  <!-- When swapping a dummy assembly with a real part, -->
-  <!-- update the include + macro call above, and adjust -->
-  <!-- parent/child link names in the mount joint below. -->
   <joint name="Revolute_3" type="continuous">
     <parent link="L110I_shoulder_2"/>
@@ -42,11 +41,34 @@
     <limit effort="100.0" velocity="1.00"/>
   </joint>
-  <!-- ROS 2 control: generated generic system -->
+  <!-- Unified 6-DoF ros2_control System -->
   <ros2_control name="Robot_to_URDF_New_Pakka_system" type="system">
     <hardware>
-      <plugin>mock_components/GenericSystem</plugin>
-      <param name="cmd_topic">sim/Robot_to_URDF_New_Pakka_system/cmd</param>
-      <param name="state_topic">sim/Robot_to_URDF_New_Pakka_system/state</param>
+      <xacro:if value="$(arg use_gazebo)">
+        <plugin>gazebo_ros2_control/GazeboSystem</plugin>
+      </xacro:if>
+      <xacro:unless value="$(arg use_gazebo)">
+        <plugin>mock_components/GenericSystem</plugin>
+        <param name="cmd_topic">sim/Robot_to_URDF_New_Pakka_system/cmd</param>
+        <param name="state_topic">sim/Robot_to_URDF_New_Pakka_system/state</param>
+      </xacro:unless>
     </hardware>
+    <joint name="Revolute_1">
+      <command_interface name="position"/>
+      <command_interface name="velocity"/>
+      <state_interface name="position">
+        <param name="initial_value">0.0</param>
+      </state_interface>
+      <state_interface name="velocity"/>
+      <state_interface name="effort"/>
+    </joint>
+    <joint name="Revolute_2">
+      <command_interface name="position"/>
+      <command_interface name="velocity"/>
+      <state_interface name="position">
+        <param name="initial_value">0.0</param>
+      </state_interface>
+      <state_interface name="velocity"/>
+      <state_interface name="effort"/>
+    </joint>
     <joint name="Revolute_3">
       <command_interface name="position"/>
@@ -86,3 +108,50 @@
     </joint>
   </ros2_control>
+  <!-- Gazebo Physics & Plugin Integration -->
+  <xacro:if value="$(arg use_gazebo)">
+    <gazebo>
+      <plugin filename="libgazebo_ros2_control.so" name="gazebo_ros2_control">
+        <parameters>$(arg gazebo_controllers)</parameters>
+      </plugin>
+    </gazebo>
+    <gazebo reference="base_link">
+      <mu1>0.8</mu1>
+      <mu2>0.8</mu2>
+      <kp>1000000.0</kp>
+      <kd>1.0</kd>
+      <material>Gazebo/Grey</material>
+    </gazebo>
+    <gazebo reference="L110I_Shoulder">
+      <mu1>0.8</mu1>
+      <mu2>0.8</mu2>
+      <material>Gazebo/Grey</material>
+    </gazebo>
+    <gazebo reference="L110I_shoulder_2">
+      <mu1>0.8</mu1>
+      <mu2>0.8</mu2>
+      <material>Gazebo/Grey</material>
+    </gazebo>
+    <gazebo reference="J2J3_Shoulder">
+      <mu1>0.8</mu1>
+      <mu2>0.8</mu2>
+      <material>Gazebo/Grey</material>
+    </gazebo>
+    <gazebo reference="Wrist_Motor">
+      <mu1>0.8</mu1>
+      <mu2>0.8</mu2>
+      <material>Gazebo/Grey</material>
+    </gazebo>
+    <gazebo reference="L70IE_Finger">
+      <mu1>0.8</mu1>
+      <mu2>0.8</mu2>
+      <material>Gazebo/Green</material>
+    </gazebo>
+    <gazebo reference="end_effector_box_link">
+      <mu1>1.2</mu1>
+      <mu2>1.2</mu2>
+      <kp>1000000.0</kp>
+      <kd>1.0</kd>
+      <material>Gazebo/DarkGrey</material>
+    </gazebo>
+  </xacro:if>
 </robot>

File: src/Robot_to_URDF_New_Pakka_description/urdf/assemblies/Robot_Assembly_URDF_New.urdf.xacro (robot description, xacro)
@@ -102,30 +102,4 @@
       <limit effort="100.0" velocity="1.00"/>
     </joint>
-    <!-- ROS 2 control: generated generic system -->
-    <ros2_control name="${prefix}Robot_Assembly_URDF_New_system" type="system">
-      <hardware>
-        <plugin>mock_components/GenericSystem</plugin>
-        <param name="cmd_topic">sim/Robot_Assembly_URDF_New_system/cmd</param>
-        <param name="state_topic">sim/Robot_Assembly_URDF_New_system/state</param>
-      </hardware>
-      <joint name="${prefix}Revolute_1">
-        <command_interface name="position"/>
-        <command_interface name="velocity"/>
-        <state_interface name="position">
-          <param name="initial_value">0.0</param>
-        </state_interface>
-        <state_interface name="velocity"/>
-        <state_interface name="effort"/>
-      </joint>
-      <joint name="${prefix}Revolute_2">
-        <command_interface name="position"/>
-        <command_interface name="velocity"/>
-        <state_interface name="position">
-          <param name="initial_value">0.0</param>
-        </state_interface>
-        <state_interface name="velocity"/>
-        <state_interface name="effort"/>
-      </joint>
-    </ros2_control>
   </xacro:macro>
 </robot>

Commit message: feat: Gazebo physics simulation pipeline with full 6-DoF peel & place benchmark suite

File: src/Robot_to_URDF_New_Pakka_description/urdf/Robot_to_URDF_New_Pakka.urdf.xacro (robot description, xacro)
@@ -1,8 +1,6 @@
 <?xml version="1.0"?>
 <robot xmlns:xacro="http://www.ros.org/wiki/xacro" name="Robot_to_URDF_New_Pakka">
-  <!-- Arguments for simulation and hardware switching -->
   <xacro:arg name="use_gazebo" default="false"/>
   <xacro:arg name="gazebo_controllers" default="$(find kerabot_moveit_config)/config/ros2_controllers.yaml"/>
-  <!-- Materials (shared across all assemblies) -->
   <material name="Steel">
     <color rgba="0.541 0.596 0.749 1.0"/>
@@ -11,13 +9,18 @@
     <color rgba="0.541 0.596 0.749 1.0"/>
   </material>
-  <!-- Assembly includes -->
+  <xacro:if value="$(arg use_gazebo)">
+    <link name="world"/>
+    <joint name="world_to_base_link" type="fixed">
+      <parent link="world"/>
+      <child link="base_link"/>
+      <origin xyz="0 0 0" rpy="0 0 0"/>
+    </joint>
+  </xacro:if>
   <xacro:include filename="$(find Robot_to_URDF_New_Pakka_description)/urdf/assemblies/J3J4_Elbow.urdf.xacro"/>
   <xacro:include filename="$(find Robot_to_URDF_New_Pakka_description)/urdf/assemblies/J6_holder.urdf.xacro"/>
   <xacro:include filename="$(find Robot_to_URDF_New_Pakka_description)/urdf/assemblies/Robot_Assembly_URDF_New.urdf.xacro"/>
-  <!-- Instantiate assemblies -->
   <xacro:J3J4_Elbow prefix=""/>
   <xacro:J6_holder prefix=""/>
   <xacro:Robot_Assembly_URDF_New prefix=""/>
-  <!-- Mount joints (cross-assembly connections) -->
   <joint name="Revolute_3" type="continuous">
     <parent link="L110I_shoulder_2"/>
@@ -41,5 +44,4 @@
     <limit effort="100.0" velocity="1.00"/>
   </joint>
-  <!-- Unified 6-DoF ros2_control System -->
   <ros2_control name="Robot_to_URDF_New_Pakka_system" type="system">
     <hardware>
@@ -108,9 +110,10 @@
     </joint>
   </ros2_control>
-  <!-- Gazebo Physics & Plugin Integration -->
   <xacro:if value="$(arg use_gazebo)">
     <gazebo>
       <plugin filename="libgazebo_ros2_control.so" name="gazebo_ros2_control">
         <parameters>$(arg gazebo_controllers)</parameters>
+        <robot_param>robot_description</robot_param>
+        <robot_param_node>robot_state_publisher</robot_param_node>
       </plugin>
     </gazebo>

File: src/Robot_to_URDF_New_Pakka_description/urdf/Robot_to_URDF_New_Pakka_gazebo.urdf (robot description, URDF)
Before this commit: robot Robot_to_URDF_New_Pakka, 7 links, 6 joints
Links:
- added link world
Joints:
- added joint world_to_base_link: type fixed, parent world, child base_link, origin xyz=0 0 0 rpy=0 0 0

File: src/Robot_to_URDF_New_Pakka_description/urdf/assemblies/J3J4_Elbow.urdf.xacro (robot description, xacro)
@@ -2,5 +2,4 @@
 <robot xmlns:xacro="http://www.ros.org/wiki/xacro" name="J3J4_Elbow_macro">
   <xacro:macro name="J3J4_Elbow" params="prefix">
-    <!-- Links -->
     <link name="${prefix}J2J3_Shoulder">
       <inertial>

File: src/Robot_to_URDF_New_Pakka_description/urdf/assemblies/J6_holder.urdf.xacro (robot description, xacro)
@@ -2,5 +2,4 @@
 <robot xmlns:xacro="http://www.ros.org/wiki/xacro" name="J6_holder_macro">
   <xacro:macro name="J6_holder" params="prefix">
-    <!-- Links -->
     <link name="${prefix}L70IE_Finger">
       <inertial>
@@ -24,7 +23,4 @@
       </collision>
     </link>
-    <!-- 6th-axis active revolute joint on the top faceplate of the L70IE_Finger motor housing.
-         - Joint origin xyz="0.150 0 0.050" places joint frame on top circular face of motor.
-         - Orientation rpy="0 1.5708 0" points local Z outward along motor face normal. -->
     <joint name="${prefix}ee_rotation_joint" type="revolute">
       <parent link="${prefix}L70IE_Finger"/>
@@ -34,7 +30,4 @@
       <limit lower="-3.14159" upper="3.14159" effort="10.0" velocity="3.14"/>
     </joint>
-    <!-- End-effector box link: 0.329 x 0.267 x 0.100 m.
-         Visual/collision offset xyz="0 0 0.050" shifts box centroid by half height (+0.050 m)
-         so the bottom 0.329 x 0.267 m face sits flush on top of the motor faceplate. -->
     <link name="${prefix}end_effector_box_link">
       <inertial>

File: src/Robot_to_URDF_New_Pakka_description/urdf/assemblies/Robot_Assembly_URDF_New.urdf.xacro (robot description, xacro)
@@ -2,5 +2,4 @@
 <robot xmlns:xacro="http://www.ros.org/wiki/xacro" name="Robot_Assembly_URDF_New_macro">
   <xacro:macro name="Robot_Assembly_URDF_New" params="prefix">
-    <!-- Links -->
     <link name="${prefix}base_link">
       <inertial>
@@ -87,5 +86,4 @@
       </collision>
     </link>
-    <!-- Joints (internal to assembly) -->
     <joint name="${prefix}Revolute_1" type="continuous">
       <parent link="${prefix}base_link"/>

Commit message: fix: joint damping and controller goal constraints for robust Gazebo trajectory execution

File: src/Robot_to_URDF_New_Pakka_description/urdf/Robot_to_URDF_New_Pakka.urdf.xacro (robot description, xacro)
@@ -29,4 +29,5 @@
     <axis xyz="-1.000000 0.000000 -0.000000"/>
     <limit effort="100.0" velocity="1.00"/>
+    <dynamics damping="2.0" friction="0.2"/>
   </joint>
   <joint name="Revolute_4" type="continuous">
@@ -36,4 +37,5 @@
     <axis xyz="-0.000000 0.000000 1.000000"/>
     <limit effort="100.0" velocity="1.00"/>
+    <dynamics damping="2.0" friction="0.2"/>
   </joint>
   <joint name="Revolute_5" type="continuous">
@@ -43,4 +45,5 @@
     <axis xyz="-0.000000 0.000000 1.000000"/>
     <limit effort="100.0" velocity="1.00"/>
+    <dynamics damping="2.0" friction="0.2"/>
   </joint>
   <ros2_control name="Robot_to_URDF_New_Pakka_system" type="system">

File: src/Robot_to_URDF_New_Pakka_description/urdf/assemblies/J6_holder.urdf.xacro (robot description, xacro)
@@ -29,4 +29,5 @@
       <axis xyz="0 0 1"/>
       <limit lower="-3.14159" upper="3.14159" effort="10.0" velocity="3.14"/>
+      <dynamics damping="1.0" friction="0.1"/>
     </joint>
     <link name="${prefix}end_effector_box_link">

File: src/Robot_to_URDF_New_Pakka_description/urdf/assemblies/Robot_Assembly_URDF_New.urdf.xacro (robot description, xacro)
@@ -92,4 +92,5 @@
       <axis xyz="0.000000 1.000000 -0.000000"/>
       <limit effort="100.0" velocity="1.00"/>
+      <dynamics damping="2.0" friction="0.2"/>
     </joint>
     <joint name="${prefix}Revolute_2" type="continuous">
@@ -99,4 +100,5 @@
       <axis xyz="0.000000 -0.000000 1.000000"/>
       <limit effort="100.0" velocity="1.00"/>
+      <dynamics damping="2.0" friction="0.2"/>
     </joint>
   </xacro:macro>
