Commit message: feat: integrate 6th-axis ee_rotation_joint and end_effector_box_link with MoveIt2 config

File: src/Robot_to_URDF_New_Pakka_description/urdf/Robot_to_URDF_New_Pakka.urdf (robot description, URDF)
Before this commit: robot Robot_to_URDF_New_Pakka, 6 links, 5 joints
Links:
- added link end_effector_box_link, mass 1.2; collision box size=0.329 0.267 0.100; visual box size=0.329 0.267 0.100
Joints:
- added joint ee_rotation_joint: type revolute, parent L70IE_Finger, child end_effector_box_link, origin xyz=0.150 0 0.050 rpy=0 1.5708 0, axis 0 0 1, limit lower=-3.14159 upper=3.14159 effort=10.0 velocity=3.14

File: src/Robot_to_URDF_New_Pakka_description/urdf/Robot_to_URDF_New_Pakka.urdf.xacro (robot description, xacro)
@@ -76,4 +76,13 @@
       <state_interface name="effort"/>
     </joint>
+    <joint name="ee_rotation_joint">
+      <command_interface name="position"/>
+      <command_interface name="velocity"/>
+      <state_interface name="position">
+        <param name="initial_value">0.0</param>
+      </state_interface>
+      <state_interface name="velocity"/>
+      <state_interface name="effort"/>
+    </joint>
   </ros2_control>
 </robot>

File: src/Robot_to_URDF_New_Pakka_description/urdf/assemblies/J6_holder.urdf.xacro (robot description, xacro)
@@ -24,4 +24,40 @@
       </collision>
     </link>
+    <!-- 6th-axis active revolute joint on the top faceplate of the L70IE_Finger motor housing.
+         - Joint origin xyz="0.150 0 0.050" places joint frame on top circular face of motor.
+         - Orientation rpy="0 1.5708 0" points local Z outward along motor face normal. -->
+    <joint name="${prefix}ee_rotation_joint" type="revolute">
+      <parent link="${prefix}L70IE_Finger"/>
+      <child link="${prefix}end_effector_box_link"/>
+      <origin xyz="0.150 0 0.050" rpy="0 1.5708 0"/>
+      <axis xyz="0 0 1"/>
+      <limit lower="-3.14159" upper="3.14159" effort="10.0" velocity="3.14"/>
+    </joint>
+    <!-- End-effector box link: 0.329 x 0.267 x 0.100 m.
+         Visual/collision offset xyz="0 0 0.050" shifts box centroid by half height (+0.050 m)
+         so the bottom 0.329 x 0.267 m face sits flush on top of the motor faceplate. -->
+    <link name="${prefix}end_effector_box_link">
+      <inertial>
+        <origin xyz="0 0 0.050" rpy="0 0 0"/>
+        <mass value="1.2"/>
+        <inertia ixx="8.129e-03" ixy="0" ixz="0"
+                 iyy="1.182e-02" iyz="0" izz="1.795e-02"/>
+      </inertial>
+      <visual>
+        <origin xyz="0 0 0.050" rpy="0 0 0"/>
+        <geometry>
+          <box size="0.329 0.267 0.100"/>
+        </geometry>
+        <material name="EE_Grey">
+          <color rgba="0.17 0.23 0.29 0.9"/>
+        </material>
+      </visual>
+      <collision>
+        <origin xyz="0 0 0.050" rpy="0 0 0"/>
+        <geometry>
+          <box size="0.329 0.267 0.100"/>
+        </geometry>
+      </collision>
+    </link>
   </xacro:macro>
 </robot>

Commit message: feat: implement collision-aware planning pipeline, fix SRDF ACM self-collisions, and add 15mm safety padding

File: src/Robot_to_URDF_New_Pakka_description/urdf/Robot_to_URDF_New_Pakka.urdf (robot description, URDF)
Before this commit: robot Robot_to_URDF_New_Pakka, 7 links, 6 joints
Links:
- link end_effector_box_link: geometry collision box size=0.359 0.297 0.130; visual box size=0.329 0.267 0.100

File: src/Robot_to_URDF_New_Pakka_description/urdf/Robot_to_URDF_New_Pakka_gazebo.urdf (robot description, URDF)
Before this commit: robot Robot_to_URDF_New_Pakka, 8 links, 7 joints
Links:
- link end_effector_box_link: geometry collision box size=0.359 0.297 0.130; visual box size=0.329 0.267 0.100

File: src/Robot_to_URDF_New_Pakka_description/urdf/assemblies/J6_holder.urdf.xacro (robot description, xacro)
@@ -50,5 +50,5 @@
         <origin xyz="0 0 0.050" rpy="0 0 0"/>
         <geometry>
-          <box size="0.329 0.267 0.100"/>
+          <box size="0.359 0.297 0.130"/>
         </geometry>
       </collision>
